Commit message: ridgeback modified

File: ridgeback_description/urdf/accessories.urdf.xacro (robot description, xacro)
@@ -14,5 +14,6 @@
   <!-- If enabled, generate the front HOKUYO UST-10LX LASER payload. -->
   <xacro:if value="$(optenv RIDGEBACK_FRONT_HOKUYO_LASER 0)">
-    <xacro:hokuyo_ust-10lx_mount prefix="front"
+    <xacro:hokuyo_ust-10lx_mount robot_name="${robot_name}"
+                                 prefix="front"
                                  topic="front/scan"
                                  location="1" />
@@ -20,5 +21,6 @@
   <!-- If enabled, generate the rear HOKUYO UST-10LX LASER payload. -->
   <xacro:if value="$(optenv RIDGEBACK_REAR_HOKUYO_LASER 0)">
-    <xacro:hokuyo_ust-10lx_mount prefix="rear"
+    <xacro:hokuyo_ust-10lx_mount robot_name="${robot_name}"
+                                 prefix="rear"
                                  topic="rear/scan"
                                  location="-1" />

File: ridgeback_description/urdf/accessories/hokuyo_ust-10lx_mount.urdf.xacro (robot description, xacro)
@@ -1,11 +1,11 @@
 <?xml version="1.0"?>
 <robot xmlns:xacro="http://www.ros.org/wiki/xacro">
-  <xacro:macro name="hokuyo_ust-10lx_mount" params="prefix topic location">
-    <joint name="${prefix}_laser_joint" type="fixed">
+  <xacro:macro name="hokuyo_ust-10lx_mount" params="robot_name prefix topic location">
+    <joint name="${robot_name}_${prefix}_laser_joint" type="fixed">
       <origin xyz="${location * 0.3932} 0 0.2330" rpy="0 0 ${PI/2 - (location * PI/2)}" />
-      <parent link="chassis_link" />
-      <child link="${prefix}_laser" />
+      <parent link="${robot_name}_chassis_link" />
+      <child link="${robot_name}_${prefix}_laser" />
     </joint>
-    <link name="${prefix}_laser">
+    <link name="${robot_name}_${prefix}_laser">
       <inertial>
         <mass value="0.130" />
@@ -30,7 +30,7 @@
       </collision>
     </link>
-    <gazebo reference="${prefix}_laser">
+    <gazebo reference="${robot_name}_${prefix}_laser">
       <turnGravityOff>false</turnGravityOff>
-      <sensor type="ray" name="${prefix}_laser">
+      <sensor type="ray" name="${robot_name}_${prefix}_laser">
         <pose>0 0 0 0 0 0</pose>
         <visualize>false</visualize>
@@ -57,6 +57,6 @@
         </ray>
         <plugin name="gazebo_ros_laser" filename="libgazebo_ros_laser.so">
-          <topicName>${topic}</topicName>
-          <frameName>${prefix}_laser</frameName>
+          <topicName>${robot_name}_${topic}</topicName>
+          <frameName>${robot_name}_${prefix}_laser</frameName>
           <hokuyoMinIntensity>101</hokuyoMinIntensity>
         </plugin>

File: ridgeback_description/urdf/ridgeback_macro.urdf.xacro (robot description, xacro)
@@ -13,5 +13,4 @@
       <limit effort="0" velocity="0" />
     </xacro:rocker>
-    <xacro:include filename="$(find ridgeback_description)/urdf/ridgeback.gazebo" />
     <xacro:include filename="$(find ridgeback_description)/urdf/accessories.urdf.xacro" />
   </xacro:macro>
