Commit message: cleaning

File: ridgeback_description/urdf/base/base.urdf.xacro (robot description, xacro)
@@ -2,13 +2,13 @@
 <robot xmlns:xacro="http://www.ros.org/wiki/xacro">
   <!-- Base -->
-  <xacro:macro name="base"  params="prefix ">
-    <link name="base_link"></link>
+  <xacro:macro name="base"  params="robot_name">
+    <link name="${robot_name}_base_link"></link>
     <!-- CHASSIS -->
-    <joint name="base_link_joint" type="fixed">
+    <joint name="${robot_name}_base_link_chasis_joint" type="fixed">
       <origin xyz="0 0 0" rpy="0 0 0" />
-      <parent link="base_link"/>
-      <child link="chassis_link" />
+      <parent link="${robot_name}_base_link"/>
+      <child link="${robot_name}_chassis_link" />
     </joint>
-    <link name="chassis_link">
+    <link name="${robot_name}_chassis_link">
       <visual>
         <origin xyz="0 0 0" rpy="0 0 0" />
@@ -18,10 +18,4 @@
         <material name="black" />
       </visual>
-      <collision>
-        <origin xyz="0 0 0"/>
-        <geometry>
-          <mesh filename="package://ridgeback_description/meshes/body-collision.stl"/>
-        </geometry>
-      </collision>
       <inertial>
         <origin xyz="0.012 0.002 0.067" rpy="${PI/2} 0 ${PI/2}"/>
@@ -33,15 +27,24 @@
       </inertial>
     </link>
-    <joint name="right_side_cover_link_joint" type="fixed">
+    <joint name="${robot_name}_right_side_cover_link_joint" type="fixed">
       <origin xyz="0 0 0" rpy="0 0 0" />
-      <parent link="chassis_link"/>
-      <child link="right_side_cover_link" />
+      <parent link="${robot_name}_chassis_link"/>
+      <child link="${robot_name}_right_side_cover_link" />
     </joint>
-    <joint name="left_side_cover_link_joint" type="fixed">
+    <link name="${robot_name}_right_side_cover_link">
+      <visual>
+        <origin xyz="0 0 0" rpy="0 0 0" />
+        <geometry>
+          <mesh filename="package://ridgeback_description/meshes/side-cover.stl"/>
+        </geometry>
+        <material name="yellow" />
+      </visual>
+    </link>
+    <joint name="${robot_name}_left_side_cover_link_joint" type="fixed">
       <origin xyz="0 0 0" rpy="0 0 0" />
-      <parent link="chassis_link"/>
-      <child link="left_side_cover_link" />
+      <parent link="${robot_name}_chassis_link"/>
+      <child link="${robot_name}_left_side_cover_link" />
     </joint>
-    <link name="left_side_cover_link">
+    <link name="${robot_name}_left_side_cover_link">
       <visual>
         <origin xyz="0 0 0" rpy="0 0 ${PI}" />
@@ -52,19 +55,10 @@
       </visual>
     </link>
-    <link name="right_side_cover_link">
-      <visual>
-        <origin xyz="0 0 0" rpy="0 0 0" />
-        <geometry>
-          <mesh filename="package://ridgeback_description/meshes/side-cover.stl"/>
-        </geometry>
-        <material name="yellow" />
-      </visual>
-    </link>
-    <joint name="front_cover_link_joint" type="fixed">
+    <joint name="${robot_name}_front_cover_link_joint" type="fixed">
       <origin xyz="0 0 0" rpy="0 0 0" />
-      <parent link="chassis_link"/>
-      <child link="front_cover_link" />
+      <parent link="${robot_name}_chassis_link"/>
+      <child link="${robot_name}_front_cover_link" />
     </joint>
-    <link name="front_cover_link">
+    <link name="${robot_name}_front_cover_link">
       <visual>
         <origin xyz="0 0 0" rpy="0 0 0" />
@@ -75,10 +69,10 @@
       </visual>
     </link>
-    <joint name="rear_cover_link_joint" type="fixed">
+    <joint name="${robot_name}_rear_cover_link_joint" type="fixed">
       <origin xyz="0 0 0" rpy="0 0 0" />
-      <parent link="chassis_link"/>
-      <child link="rear_cover_link" />
+      <parent link="${robot_name}_chassis_link"/>
+      <child link="${robot_name}_rear_cover_link" />
     </joint>
-    <link name="rear_cover_link">
+    <link name="${robot_name}_rear_cover_link">
       <visual>
         <origin xyz="0 0 0" rpy="0 0 ${PI}" />
@@ -89,15 +83,10 @@
       </visual>
     </link>
-    <joint name="front_lights_link_joint" type="fixed">
+    <joint name="${robot_name}_front_lights_link_joint" type="fixed">
       <origin xyz="0 0 0" rpy="0 0 0" />
-      <parent link="chassis_link"/>
-      <child link="front_lights_link" />
+      <parent link="${robot_name}_chassis_link"/>
+      <child link="${robot_name}_front_lights_link" />
     </joint>
-    <joint name="rear_lights_link_joint" type="fixed">
-      <origin xyz="0 0 0" rpy="0 0 0" />
-      <parent link="chassis_link"/>
-      <child link="rear_lights_link" />
-    </joint>
-    <link name="front_lights_link">
+    <link name="${robot_name}_front_lights_link">
       <visual>
         <origin xyz="0 0 0" rpy="0 0 0" />
@@ -108,5 +97,10 @@
       </visual>
     </link>
-    <link name="rear_lights_link">
+    <joint name="${robot_name}_rear_lights_link_joint" type="fixed">
+      <origin xyz="0 0 0" rpy="0 0 0" />
+      <parent link="${robot_name}_chassis_link"/>
+      <child link="${robot_name}_rear_lights_link" />
+    </joint>
+    <link name="${robot_name}_rear_lights_link">
       <visual>
         <origin xyz="0 0 0" rpy="0 0 ${PI}" />
@@ -117,10 +111,10 @@
       </visual>
     </link>
-    <joint name="top_link_joint" type="fixed">
+    <joint name="${robot_name}_top_link_joint" type="fixed">
       <origin xyz="0 0 0" rpy="0 0 0" />
-      <parent link="chassis_link"/>
-      <child link="top_link" />
+      <parent link="${robot_name}_chassis_link"/>
+      <child link="${robot_name}_top_link" />
     </joint>
-    <link name="top_link">
+    <link name="${robot_name}_top_link">
       <visual>
         <origin xyz="0 0 0" rpy="0 0 0" />
@@ -130,17 +124,11 @@
         <material name="black" />
       </visual>
-      <collision>
-        <origin xyz="0 0 0" rpy="0 0 0" />
-        <geometry>
-          <mesh filename="package://ridgeback_description/meshes/top.stl"/>
-        </geometry>
-      </collision>
     </link>
-    <joint name="axle_joint" type="fixed">
+    <joint name="${robot_name}_axle_joint" type="fixed">
       <origin xyz="0 0 ${axle_offset}" rpy="0 0 0" />
-      <parent link="chassis_link"/>
-      <child link="axle_link" />
+      <parent link="${robot_name}_chassis_link"/>
+      <child link="${robot_name}_axle_link" />
     </joint>
-    <link name="axle_link">
+    <link name="${robot_name}_axle_link">
       <visual>
         <origin xyz="0 0 0" rpy="0 ${PI/2} 0" />
@@ -151,11 +139,11 @@
       </visual>
     </link>
-    <link name="mid_mount" />
+    <link name="${robot_name}_mid_mount" />
     <joint name="mid_mount_joint" type="fixed">
-      <parent link="base_link" />
-      <child link="mid_mount" />
+      <parent link="${robot_name}_base_link" />
+      <child link="${robot_name}_mid_mount" />
       <origin xyz="0 0 ${deck_height}" rpy="0 0 0"/>
     </joint>
-    <link name="imu_link">
+    <link name="${robot_name}_imu_link">
       <inertial>
         <mass value="0.001"/>
@@ -164,7 +152,7 @@
       </inertial>
     </link>
-    <joint name="imu_joint" type="fixed">
-      <parent link="chassis_link" />
-      <child link="imu_link" />
+    <joint name="${robot_name}_imu_joint" type="fixed">
+      <parent link="${robot_name}_chassis_link" />
+      <child link="${robot_name}_imu_link" />
       <origin xyz="${imu_offset_x} ${imu_offset_y} ${imu_offset_z}" rpy="0 0 0"/>
     </joint>

File: ridgeback_description/urdf/ridgeback.urdf.xacro (robot description, xacro)
@@ -25,6 +25,9 @@
   <xacro:include filename="$(find ridgeback_description)/urdf/rocker/rocker.urdf.xacro"/>
   <xacro:include filename="$(find ridgeback_description)/urdf/wheel/wheel.urdf.xacro"/>
-  <xacro:include filename="$(find cri_efe_aruco)/urdf/single_markers/marker_6.urdf.xacro"/>
-  <xacro:include filename="$(find cri_efe_aruco)/urdf/multi_markers/multi_marker_0.urdf.xacro"/>
+  <!--xacro:include filename="$(find cri_efe_aruco)/urdf/multi_markers/multi_marker_0.urdf.xacro"/>
+  <xacro:include filename="$(find cri_efe_aruco)/urdf/multi_markers/multi_marker_1.urdf.xacro"/>
+  -->
+  <xacro:include filename="$(find cri_efe_aruco)/urdf/multi_markers/quad_marker_0.urdf.xacro"/>
+  <xacro:include filename="$(find cri_efe_aruco)/urdf/multi_markers/quad_marker_1.urdf.xacro"/>
   <xacro:base prefix=""/>
   <xacro:rocker prefix="front" joint_type="revolute" location="1" >
@@ -34,10 +37,8 @@
     <limit effort="0" velocity="0" />
   </xacro:rocker>
-  <xacro:multi_marker_0 pad_base="top_link" x="0.2" y="-0.2" z="0.29" yaw="0.0" scale="0.9"/>
+  <xacro:quad_marker_0 pad_base="top_link" x="0.25" y="-0.25" z="0.29" yaw="0.0" scale="1.2"/>
+  <xacro:quad_marker_1 pad_base="top_link" x="0.25" y="0.25" z="0.29" yaw="0.0" scale="1.2"/>
   <!-- Bring in simulation data for Gazebo. -->
   <xacro:include filename="$(find ridgeback_description)/urdf/ridgeback.gazebo" />
-  <xacro:if value="${simulation}">
-    <xacro:include filename="$(find cri_efe_description)/urdf/include/ridgeback_plugin.gazebo.xacro" />
-  </xacro:if>
   <xacro:include filename="$(find ridgeback_description)/urdf/accessories.urdf.xacro" />
   <xacro:include filename="$(optenv RIDGEBACK_URDF_EXTRAS empty.urdf)" />

File: ridgeback_description/urdf/rocker/rocker.urdf.xacro (robot description, xacro)
@@ -1,7 +1,7 @@
 <?xml version="1.0"?>
 <robot xmlns:xacro="http://www.ros.org/wiki/xacro">
-  <!-- Base -->
-  <xacro:macro name="rocker"  params="prefix joint_type location *joint_limits">
-    <link name="${prefix}_rocker_link">
+  <!-- ROCKER -->
+  <xacro:macro name="rocker"  params="robot_name prefix joint_type location *joint_limits">
+    <link name="${robot_name}_${prefix}_rocker_link">
       <visual>
         <origin xyz="0 0 0" rpy="${PI/2} 0 ${PI/2}" />
@@ -20,15 +20,16 @@
       </inertial>
     </link>
-    <joint name="${prefix}_rocker" type="${joint_type}">
-      <parent link="axle_link"/>
-      <child link="${prefix}_rocker_link" />
+    <joint name="${robot_name}_${prefix}_rocker" type="${joint_type}">
+      <parent link="${robot_name}_axle_link"/>
+      <child link="${robot_name}_${prefix}_rocker_link" />
       <origin xyz="${location*rocker_offset} 0 0" rpy="0 0 0" />
       <axis xyz="1 0 0" />
       <xacro:insert_block name="joint_limits" />
     </joint>
-    <xacro:wheel prefix="${prefix}" side="left">
+    <!-- WHEELS-->
+    <xacro:wheel robot_name="${robot_name}" prefix="${prefix}" side="left">
       <origin xyz="0 ${rocker_width/2 + wheel_width/2} 0" rpy="0 0 0" />
     </xacro:wheel>
-    <xacro:wheel prefix="${prefix}" side="right">
+    <xacro:wheel robot_name="${robot_name}" prefix="${prefix}" side="right">
       <origin xyz="0 ${-(rocker_width/2 + wheel_width/2)} 0" rpy="0 0 0" />
     </xacro:wheel>

File: ridgeback_description/urdf/wheel/wheel.urdf.xacro (robot description, xacro)
@@ -2,6 +2,6 @@
 <robot xmlns:xacro="http://www.ros.org/wiki/xacro">
   <!-- Base -->
-  <xacro:macro name="wheel"  params="prefix side *joint_pose">
-    <link name="${prefix}_${side}_wheel_link">
+  <xacro:macro name="wheel"  params="robot_name prefix side *joint_pose">
+    <link name="${robot_name}_${prefix}_${side}_wheel_link">
       <visual>
         <origin xyz="0 0 0" rpy="${PI/2} 0 0"/>
@@ -26,16 +26,16 @@
       </inertial>
     </link>
-    <joint name="${prefix}_${side}_wheel" type="continuous">
-      <parent link="${prefix}_rocker_link"/>
-      <child link="${prefix}_${side}_wheel_link" />
+    <joint name="${robot_name}_${prefix}_${side}_wheel" type="continuous">
+      <parent link="${robot_name}_${prefix}_rocker_link"/>
+      <child link="${robot_name}_${prefix}_${side}_wheel_link" />
       <xacro:insert_block name="joint_pose" />
       <axis xyz="0 1 0" />
     </joint>
-    <transmission name="${prefix}_wheel_trans">
+    <transmission name="${robot_name}_${prefix}_wheel_trans">
       <type>transmission_interface/SimpleTransmission</type>
-      <joint name="${prefix}_${side}_wheel">
+      <joint name="${robot_name}_${prefix}_${side}_wheel">
         <hardwareInterface>hardware_interface/VelocityJointInterface</hardwareInterface>
       </joint>
-      <actuator name="${prefix}_${side}_actuator">
+      <actuator name="${robot_name}_${prefix}_${side}_actuator">
         <mechanicalReduction>1</mechanicalReduction>
       </actuator>
